Commit message: Replace all files with final_robin content

File: install/roverrobotics_description/share/roverrobotics_description/urdf/accessories/rplidar_s2.urdf (robot description, URDF)
Before this commit: robot rplidar_s2, 1 links, 1 joints
Joints:
- joint lidar_to_payload: origin xyz=0.174 0 0.10 rpy=0 0 3.1415 -> xyz=0.174 0 0.145 rpy=0 0 3.1415

File: install/roverrobotics_description/share/roverrobotics_description/urdf/max_150.urdf (robot description, URDF)
Before this commit: robot rover_max, 6 links, 5 joints
Joints:
- joint base_to_chassis: origin xyz=0 0 0.165 -> xyz=0 0 0.1645

File: install/roverrobotics_description/share/roverrobotics_description/urdf/miti_65.urdf (robot description, URDF)
Before this commit: robot rover_miti, 6 links, 5 joints
Joints:
- joint base_to_chassis: origin xyz=0 0 0.061 -> xyz=0 0 0.062
